File: PCB/aniboard.kicad_pcb (KiCad board)
At the start: 2 copper layers, 1 part, among them U1 Pico

Commit message: First three rows
Parts:
- added S1: MX_stab, PCM_marbastlib-mx:STAB_MX_P_2u, F.Cu at (281.0, 45.2)
- added SW1: SW_Push, PCM_marbastlib-mx:SW_MX_1.5u, F.Cu at (28.6, 26.2)
- added SW10: SW_Push, PCM_marbastlib-mx:SW_MX_1u, F.Cu at (204.8, 26.2)
- added SW11: SW_Push, PCM_marbastlib-mx:SW_MX_1u, F.Cu at (223.8, 26.2)
- added SW12: SW_Push, PCM_marbastlib-mx:SW_MX_1u, F.Cu at (242.9, 26.2)
- added SW13: SW_Push, PCM_marbastlib-mx:SW_MX_1u, F.Cu at (261.9, 26.2)
- added SW14: SW_Push, PCM_marbastlib-mx:SW_MX_1.5u, F.Cu at (285.8, 26.2)
- added SW15: SW_Push, PCM_marbastlib-mx:SW_MX_1u, F.Cu at (23.8, 45.2)
- added SW16: SW_Push, PCM_marbastlib-mx:SW_MX_1u, F.Cu at (42.9, 45.2)
- added SW17: SW_Push, PCM_marbastlib-mx:SW_MX_1u, F.Cu at (61.9, 45.2)
- added SW18: SW_Push, PCM_marbastlib-mx:SW_MX_1u, F.Cu at (81.0, 45.2)
- added SW19: SW_Push, PCM_marbastlib-mx:SW_MX_1u, F.Cu at (100.0, 45.2)
- added SW2: SW_Push, PCM_marbastlib-mx:SW_MX_1u, F.Cu at (52.4, 26.2)
- added SW20: SW_Push, PCM_marbastlib-mx:SW_MX_1u, F.Cu at (119.1, 45.2)
- added SW21: SW_Push, PCM_marbastlib-mx:SW_MX_1u, F.Cu at (138.1, 45.2)
- added SW22: SW_Push, PCM_marbastlib-mx:SW_MX_1u, F.Cu at (157.2, 45.2)
- added SW23: SW_Push, PCM_marbastlib-mx:SW_MX_1u, F.Cu at (176.2, 45.2)
- added SW24: SW_Push, PCM_marbastlib-mx:SW_MX_1u, F.Cu at (195.3, 45.2)
- added SW25: SW_Push, PCM_marbastlib-mx:SW_MX_1u, F.Cu at (214.3, 45.2)
- added SW26: SW_Push, PCM_marbastlib-mx:SW_MX_1u, F.Cu at (233.4, 45.2)
- added SW27: SW_Push, PCM_marbastlib-mx:SW_MX_1u, F.Cu at (252.4, 45.2)
- added SW28: SW_Push, PCM_marbastlib-mx:SW_MX_1u, F.Cu at (281.0, 45.2)
- added SW29: SW_Push, PCM_marbastlib-mx:SW_MX_1.5u, F.Cu at (28.6, 64.3)
- added SW3: SW_Push, PCM_marbastlib-mx:SW_MX_1u, F.Cu at (71.4, 26.2)
- added SW30: SW_Push, PCM_marbastlib-mx:SW_MX_1u, F.Cu at (52.4, 64.3)
- added SW31: SW_Push, PCM_marbastlib-mx:SW_MX_1u, F.Cu at (71.4, 64.3)
- added SW32: SW_Push, PCM_marbastlib-mx:SW_MX_1u, F.Cu at (90.5, 64.3)
- added SW33: SW_Push, PCM_marbastlib-mx:SW_MX_1u, F.Cu at (109.5, 64.3)
- added SW34: SW_Push, PCM_marbastlib-mx:SW_MX_1u, F.Cu at (128.6, 64.3)
- added SW35: SW_Push, PCM_marbastlib-mx:SW_MX_1u, F.Cu at (147.6, 64.3)
- added SW36: SW_Push, PCM_marbastlib-mx:SW_MX_1u, F.Cu at (166.7, 64.3)
- added SW37: SW_Push, PCM_marbastlib-mx:SW_MX_1u, F.Cu at (185.7, 64.3)
- added SW38: SW_Push, PCM_marbastlib-mx:SW_MX_1u, F.Cu at (204.8, 64.3)
- added SW39: SW_Push, PCM_marbastlib-mx:SW_MX_1u, F.Cu at (223.8, 64.3)
- added SW4: SW_Push, PCM_marbastlib-mx:SW_MX_1u, F.Cu at (90.5, 26.2)
- added SW40: SW_Push, PCM_marbastlib-mx:SW_MX_1u, F.Cu at (242.9, 64.3)
- added SW41: SW_Push, PCM_marbastlib-mx:SW_MX_1u, F.Cu at (261.9, 64.3)
- added SW42: SW_Push, PCM_marbastlib-mx:SW_MX_1.5u, F.Cu at (285.8, 64.3)
- added SW5: SW_Push, PCM_marbastlib-mx:SW_MX_1u, F.Cu at (109.5, 26.2)
- added SW6: SW_Push, PCM_marbastlib-mx:SW_MX_1u, F.Cu at (128.6, 26.2)
- added SW7: SW_Push, PCM_marbastlib-mx:SW_MX_1u, F.Cu at (147.6, 26.2)
- added SW8: SW_Push, PCM_marbastlib-mx:SW_MX_1u, F.Cu at (166.7, 26.2)
- added SW9: SW_Push, PCM_marbastlib-mx:SW_MX_1u, F.Cu at (185.7, 26.2)
- moved U1 102.3 mm to (37.5, 161.4)

Commit message: Keyboard layout
Parts:
- added S2: MX_stab, PCM_marbastlib-mx:STAB_MX_2.25u, F.Cu at (278.6, 83.3)
- added S3: MX_stab, PCM_marbastlib-mx:STAB_MX_2.25u, F.Cu at (35.7, 102.4)
- added S4: MX_stab, PCM_marbastlib-mx:STAB_MX_2.75u, F.Cu at (273.8, 102.4)
- added S5: MX_stab, PCM_marbastlib-mx:STAB_MX_6.25u, F.Cu at (145.3, 121.4)
- added SW43: SW_Push, PCM_marbastlib-mx:SW_MX_1.75u, F.Cu at (31.0, 83.3)
- added SW44: SW_Push, PCM_marbastlib-mx:SW_MX_1u, F.Cu at (57.1, 83.3)
- added SW45: SW_Push, PCM_marbastlib-mx:SW_MX_1u, F.Cu at (76.2, 83.3)
- added SW46: SW_Push, PCM_marbastlib-mx:SW_MX_1u, F.Cu at (95.2, 83.3)
- added SW47: SW_Push, PCM_marbastlib-mx:SW_MX_1u, F.Cu at (114.3, 83.3)
- added SW48: SW_Push, PCM_marbastlib-mx:SW_MX_1u, F.Cu at (133.3, 83.3)
- added SW49: SW_Push, PCM_marbastlib-mx:SW_MX_1u, F.Cu at (152.4, 83.3)
- added SW50: SW_Push, PCM_marbastlib-mx:SW_MX_1u, F.Cu at (171.4, 83.3)
- added SW51: SW_Push, PCM_marbastlib-mx:SW_MX_1u, F.Cu at (190.5, 83.3)
- added SW52: SW_Push, PCM_marbastlib-mx:SW_MX_1u, F.Cu at (209.6, 83.3)
- added SW53: SW_Push, PCM_marbastlib-mx:SW_MX_1u, F.Cu at (228.6, 83.3)
- added SW54: SW_Push, PCM_marbastlib-mx:SW_MX_1u, F.Cu at (247.7, 83.3)
- added SW55: SW_Push, PCM_marbastlib-mx:SW_MX_1u, F.Cu at (278.6, 83.3)
- added SW56: SW_Push, PCM_marbastlib-mx:SW_MX_1u, F.Cu at (35.7, 102.4)
- added SW57: SW_Push, PCM_marbastlib-mx:SW_MX_1u, F.Cu at (66.7, 102.4)
- added SW58: SW_Push, PCM_marbastlib-mx:SW_MX_1u, F.Cu at (85.7, 102.4)
- added SW59: SW_Push, PCM_marbastlib-mx:SW_MX_1u, F.Cu at (104.8, 102.4)
- added SW60: SW_Push, PCM_marbastlib-mx:SW_MX_1u, F.Cu at (123.8, 102.4)
- added SW61: SW_Push, PCM_marbastlib-mx:SW_MX_1u, F.Cu at (142.9, 102.4)
- added SW62: SW_Push, PCM_marbastlib-mx:SW_MX_1u, F.Cu at (161.9, 102.4)
- added SW63: SW_Push, PCM_marbastlib-mx:SW_MX_1u, F.Cu at (181.0, 102.4)
- added SW64: SW_Push, PCM_marbastlib-mx:SW_MX_1u, F.Cu at (200.0, 102.4)
- added SW65: SW_Push, PCM_marbastlib-mx:SW_MX_1u, F.Cu at (219.1, 102.4)
- added SW66: SW_Push, PCM_marbastlib-mx:SW_MX_1u, F.Cu at (238.1, 102.4)
- added SW67: SW_Push, PCM_marbastlib-mx:SW_MX_1u, F.Cu at (273.8, 102.4)
- added SW68: SW_Push, PCM_marbastlib-mx:SW_MX_1.25u, F.Cu at (26.2, 121.4)
- added SW69: SW_Push, PCM_marbastlib-mx:SW_MX_1.25u, F.Cu at (50.0, 121.4)
- added SW70: SW_Push, PCM_marbastlib-mx:SW_MX_1.25u, F.Cu at (73.8, 121.4)
- added SW71: SW_Push, PCM_marbastlib-mx:SW_MX_1u, F.Cu at (145.3, 121.4)
- added SW72: SW_Push, PCM_marbastlib-mx:SW_MX_1.25u, F.Cu at (216.7, 121.4)
- added SW73: SW_Push, PCM_marbastlib-mx:SW_MX_1.25u, F.Cu at (240.5, 121.4)
- added SW74: SW_Push, PCM_marbastlib-mx:SW_MX_1.25u, F.Cu at (264.3, 121.4)
- added SW75: SW_Push, PCM_marbastlib-mx:SW_MX_1.25u, F.Cu at (288.1, 121.4)
- added SW76: SW_Push, PCM_marbastlib-mx:SW_MX_1u, F.Cu at (314.3, 121.4)
- added SW77: SW_Push, PCM_marbastlib-mx:SW_MX_1u, F.Cu at (333.4, 121.4)
- added SW78: SW_Push, PCM_marbastlib-mx:SW_MX_1u, F.Cu at (352.4, 121.4)
- added SW79: SW_Push, PCM_marbastlib-mx:SW_MX_1u, F.Cu at (333.4, 102.4)
- added SW80: SW_Push, PCM_marbastlib-mx:SW_MX_1u, F.Cu at (314.3, 45.2)
- added SW81: SW_Push, PCM_marbastlib-mx:SW_MX_1u, F.Cu at (333.4, 45.2)
- added SW82: SW_Push, PCM_marbastlib-mx:SW_MX_1u, F.Cu at (352.4, 45.2)
- added SW83: SW_Push, PCM_marbastlib-mx:SW_MX_1u, F.Cu at (314.3, 64.3)
- added SW84: SW_Push, PCM_marbastlib-mx:SW_MX_1u, F.Cu at (333.4, 64.3)
- added SW85: SW_Push, PCM_marbastlib-mx:SW_MX_1u, F.Cu at (352.4, 64.3)
- added SW86: SW_Push, PCM_marbastlib-mx:SW_MX_1u, F.Cu at (314.3, 83.3)
- added SW87: SW_Push, PCM_marbastlib-mx:SW_MX_1u, F.Cu at (333.4, 83.3)
- added SW88: SW_Push, PCM_marbastlib-mx:SW_MX_1u, F.Cu at (352.4, 83.3)
- S1: footprint PCM_marbastlib-mx:STAB_MX_P_2u -> PCM_marbastlib-mx:STAB_MX_2u
- moved U1 69.6 mm to (106.5, 170.0)

Commit message: Continue routing PCB
Parts:
- added D1: D, Diode_THT:D_DO-35_SOD27_P7.62mm_Horizontal, F.Cu at (185.6, 164.4)
- added D10: D, Diode_THT:D_DO-35_SOD27_P7.62mm_Horizontal, F.Cu at (185.6, 196.3)
- added D11: D, Diode_THT:D_DO-35_SOD27_P7.62mm_Horizontal, F.Cu at (185.6, 199.9)
- added D12: D, Diode_THT:D_DO-35_SOD27_P7.62mm_Horizontal, F.Cu at (185.6, 203.4)
- added D13: D, Diode_THT:D_DO-35_SOD27_P7.62mm_Horizontal, F.Cu at (185.6, 207.0)
- added D14: D, Diode_THT:D_DO-35_SOD27_P7.62mm_Horizontal, F.Cu at (185.6, 210.6)
- added D15: D, Diode_THT:D_DO-35_SOD27_P7.62mm_Horizontal, F.Cu at (185.6, 214.1)
- added D16: D, Diode_THT:D_DO-35_SOD27_P7.62mm_Horizontal, F.Cu at (185.6, 217.7)
- added D17: D, Diode_THT:D_DO-35_SOD27_P7.62mm_Horizontal, F.Cu at (185.6, 221.2)
- added D18: D, Diode_THT:D_DO-35_SOD27_P7.62mm_Horizontal, F.Cu at (185.6, 224.8)
- added D19: D, Diode_THT:D_DO-35_SOD27_P7.62mm_Horizontal, F.Cu at (196.4, 164.4)
- added D2: D, Diode_THT:D_DO-35_SOD27_P7.62mm_Horizontal, F.Cu at (185.6, 167.9)
- added D20: D, Diode_THT:D_DO-35_SOD27_P7.62mm_Horizontal, F.Cu at (196.4, 167.9)
- added D21: D, Diode_THT:D_DO-35_SOD27_P7.62mm_Horizontal, F.Cu at (196.4, 171.5)
- added D22: D, Diode_THT:D_DO-35_SOD27_P7.62mm_Horizontal, F.Cu at (196.4, 175.1)
- added D23: D, Diode_THT:D_DO-35_SOD27_P7.62mm_Horizontal, F.Cu at (196.4, 178.6)
- added D24: D, Diode_THT:D_DO-35_SOD27_P7.62mm_Horizontal, F.Cu at (196.4, 182.2)
- added D25: D, Diode_THT:D_DO-35_SOD27_P7.62mm_Horizontal, F.Cu at (196.4, 185.7)
- added D26: D, Diode_THT:D_DO-35_SOD27_P7.62mm_Horizontal, F.Cu at (196.4, 189.2)
- added D27: D, Diode_THT:D_DO-35_SOD27_P7.62mm_Horizontal, F.Cu at (196.4, 192.8)
- added D28: D, Diode_THT:D_DO-35_SOD27_P7.62mm_Horizontal, F.Cu at (196.4, 196.3)
- added D29: D, Diode_THT:D_DO-35_SOD27_P7.62mm_Horizontal, F.Cu at (196.4, 199.9)
- added D3: D, Diode_THT:D_DO-35_SOD27_P7.62mm_Horizontal, F.Cu at (185.6, 171.5)
- added D30: D, Diode_THT:D_DO-35_SOD27_P7.62mm_Horizontal, F.Cu at (196.4, 203.4)
- added D31: D, Diode_THT:D_DO-35_SOD27_P7.62mm_Horizontal, F.Cu at (196.4, 207.0)
- added D32: D, Diode_THT:D_DO-35_SOD27_P7.62mm_Horizontal, F.Cu at (196.4, 210.6)
- added D33: D, Diode_THT:D_DO-35_SOD27_P7.62mm_Horizontal, F.Cu at (196.4, 214.1)
- added D34: D, Diode_THT:D_DO-35_SOD27_P7.62mm_Horizontal, F.Cu at (196.4, 217.7)
- added D35: D, Diode_THT:D_DO-35_SOD27_P7.62mm_Horizontal, F.Cu at (196.4, 221.2)
- added D36: D, Diode_THT:D_DO-35_SOD27_P7.62mm_Horizontal, F.Cu at (196.4, 224.8)
- added D37: D, Diode_THT:D_DO-35_SOD27_P7.62mm_Horizontal, F.Cu at (207.2, 164.4)
- added D38: D, Diode_THT:D_DO-35_SOD27_P7.62mm_Horizontal, F.Cu at (207.2, 167.9)
- added D39: D, Diode_THT:D_DO-35_SOD27_P7.62mm_Horizontal, F.Cu at (207.2, 171.5)
- added D4: D, Diode_THT:D_DO-35_SOD27_P7.62mm_Horizontal, F.Cu at (185.6, 175.1)
- added D40: D, Diode_THT:D_DO-35_SOD27_P7.62mm_Horizontal, F.Cu at (207.2, 175.1)
- added D41: D, Diode_THT:D_DO-35_SOD27_P7.62mm_Horizontal, F.Cu at (207.2, 178.6)
- added D42: D, Diode_THT:D_DO-35_SOD27_P7.62mm_Horizontal, F.Cu at (207.2, 182.2)
- added D43: D, Diode_THT:D_DO-35_SOD27_P7.62mm_Horizontal, F.Cu at (207.2, 185.7)
- added D44: D, Diode_THT:D_DO-35_SOD27_P7.62mm_Horizontal, F.Cu at (207.2, 189.2)
- added D45: D, Diode_THT:D_DO-35_SOD27_P7.62mm_Horizontal, F.Cu at (207.2, 192.8)
- added D46: D, Diode_THT:D_DO-35_SOD27_P7.62mm_Horizontal, F.Cu at (207.2, 196.3)
- added D47: D, Diode_THT:D_DO-35_SOD27_P7.62mm_Horizontal, F.Cu at (207.2, 199.9)
- added D48: D, Diode_THT:D_DO-35_SOD27_P7.62mm_Horizontal, F.Cu at (207.2, 203.4)
- added D49: D, Diode_THT:D_DO-35_SOD27_P7.62mm_Horizontal, F.Cu at (207.2, 207.0)
- added D5: D, Diode_THT:D_DO-35_SOD27_P7.62mm_Horizontal, F.Cu at (185.6, 178.6)
- added D50: D, Diode_THT:D_DO-35_SOD27_P7.62mm_Horizontal, F.Cu at (207.2, 210.6)
- added D51: D, Diode_THT:D_DO-35_SOD27_P7.62mm_Horizontal, F.Cu at (207.2, 214.1)
- added D52: D, Diode_THT:D_DO-35_SOD27_P7.62mm_Horizontal, F.Cu at (207.2, 217.7)
- added D53: D, Diode_THT:D_DO-35_SOD27_P7.62mm_Horizontal, F.Cu at (207.2, 221.2)
- added D54: D, Diode_THT:D_DO-35_SOD27_P7.62mm_Horizontal, F.Cu at (207.2, 224.8)
- added D55: D, Diode_THT:D_DO-35_SOD27_P7.62mm_Horizontal, F.Cu at (217.9, 164.4)
- added D56: D, Diode_THT:D_DO-35_SOD27_P7.62mm_Horizontal, F.Cu at (217.9, 167.9)
- added D57: D, Diode_THT:D_DO-35_SOD27_P7.62mm_Horizontal, F.Cu at (217.9, 171.5)
- added D58: D, Diode_THT:D_DO-35_SOD27_P7.62mm_Horizontal, F.Cu at (217.9, 175.1)
- added D59: D, Diode_THT:D_DO-35_SOD27_P7.62mm_Horizontal, F.Cu at (217.9, 178.6)
- added D6: D, Diode_THT:D_DO-35_SOD27_P7.62mm_Horizontal, F.Cu at (185.6, 182.2)
- added D60: D, Diode_THT:D_DO-35_SOD27_P7.62mm_Horizontal, F.Cu at (217.9, 182.2)
- added D61: D, Diode_THT:D_DO-35_SOD27_P7.62mm_Horizontal, F.Cu at (217.9, 185.7)
- added D62: D, Diode_THT:D_DO-35_SOD27_P7.62mm_Horizontal, F.Cu at (217.9, 189.2)
- added D63: D, Diode_THT:D_DO-35_SOD27_P7.62mm_Horizontal, F.Cu at (217.9, 192.8)
- added D64: D, Diode_THT:D_DO-35_SOD27_P7.62mm_Horizontal, F.Cu at (217.9, 196.3)
- added D65: D, Diode_THT:D_DO-35_SOD27_P7.62mm_Horizontal, F.Cu at (217.9, 199.9)
- added D66: D, Diode_THT:D_DO-35_SOD27_P7.62mm_Horizontal, F.Cu at (217.9, 203.4)
- added D67: D, Diode_THT:D_DO-35_SOD27_P7.62mm_Horizontal, F.Cu at (217.9, 207.0)
- added D68: D, Diode_THT:D_DO-35_SOD27_P7.62mm_Horizontal, F.Cu at (217.9, 210.6)
- added D69: D, Diode_THT:D_DO-35_SOD27_P7.62mm_Horizontal, F.Cu at (217.9, 214.1)
- added D7: D, Diode_THT:D_DO-35_SOD27_P7.62mm_Horizontal, F.Cu at (185.6, 185.7)
- added D70: D, Diode_THT:D_DO-35_SOD27_P7.62mm_Horizontal, F.Cu at (217.9, 217.7)
- added D71: D, Diode_THT:D_DO-35_SOD27_P7.62mm_Horizontal, F.Cu at (217.9, 221.2)
- added D72: D, Diode_THT:D_DO-35_SOD27_P7.62mm_Horizontal, F.Cu at (217.9, 224.8)
- added D73: D, Diode_THT:D_DO-35_SOD27_P7.62mm_Horizontal, F.Cu at (228.7, 164.4)
- added D74: D, Diode_THT:D_DO-35_SOD27_P7.62mm_Horizontal, F.Cu at (228.7, 167.9)
- added D75: D, Diode_THT:D_DO-35_SOD27_P7.62mm_Horizontal, F.Cu at (228.7, 171.5)
- added D76: D, Diode_THT:D_DO-35_SOD27_P7.62mm_Horizontal, F.Cu at (228.7, 175.1)
- added D77: D, Diode_THT:D_DO-35_SOD27_P7.62mm_Horizontal, F.Cu at (228.7, 178.6)
- added D78: D, Diode_THT:D_DO-35_SOD27_P7.62mm_Horizontal, F.Cu at (228.7, 182.2)
- added D79: D, Diode_THT:D_DO-35_SOD27_P7.62mm_Horizontal, F.Cu at (228.7, 185.7)
- added D8: D, Diode_THT:D_DO-35_SOD27_P7.62mm_Horizontal, F.Cu at (185.6, 189.2)
- added D80: D, Diode_THT:D_DO-35_SOD27_P7.62mm_Horizontal, F.Cu at (228.7, 189.2)
- added D81: D, Diode_THT:D_DO-35_SOD27_P7.62mm_Horizontal, F.Cu at (228.7, 192.8)
- added D82: D, Diode_THT:D_DO-35_SOD27_P7.62mm_Horizontal, F.Cu at (228.7, 196.3)
- added D83: D, Diode_THT:D_DO-35_SOD27_P7.62mm_Horizontal, F.Cu at (228.7, 199.9)
- added D84: D, Diode_THT:D_DO-35_SOD27_P7.62mm_Horizontal, F.Cu at (228.7, 203.4)
- added D85: D, Diode_THT:D_DO-35_SOD27_P7.62mm_Horizontal, F.Cu at (228.7, 207.0)
- added D86: D, Diode_THT:D_DO-35_SOD27_P7.62mm_Horizontal, F.Cu at (228.7, 210.6)
- added D87: D, Diode_THT:D_DO-35_SOD27_P7.62mm_Horizontal, F.Cu at (228.7, 214.1)
- added D88: D, Diode_THT:D_DO-35_SOD27_P7.62mm_Horizontal, F.Cu at (228.7, 217.7)
- added D9: D, Diode_THT:D_DO-35_SOD27_P7.62mm_Horizontal, F.Cu at (185.6, 192.8)
- moved U1 279.4 mm to (357.4, 47.1), turned to -90 degrees
- moved S2 30.3 mm to (299.9, 104.9)
- moved S4 30.3 mm to (295.2, 123.9)
- moved S5 30.3 mm to (166.6, 143.0)
- moved SW48 30.3 mm to (154.7, 104.9)
- moved SW50 30.3 mm to (192.8, 104.9)
- moved SW53 30.3 mm to (249.9, 104.9)
- moved SW55 30.3 mm to (299.9, 104.9)
- moved SW63 30.3 mm to (202.3, 123.9)
- moved SW65 30.3 mm to (240.4, 123.9)
- moved SW66 30.3 mm to (259.4, 123.9)
- moved SW67 30.3 mm to (295.2, 123.9)
- moved SW71 30.3 mm to (166.6, 143.0)
- moved SW72 30.3 mm to (238.0, 143.0)
- moved SW76 30.3 mm to (335.6, 143.0)
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Connections:
- SW55 pad 1: COL12 -> COL13
- SW67 pad 1: COL11 -> COL13
- SW75 pad 1: COL11 -> COL13
- U1 pad 1: unconnected-(U1-GPIO0-Pad1) -> COL0
- U1 pad 10: unconnected-(U1-GPIO7-Pad10) -> COL7
- U1 pad 11: unconnected-(U1-GPIO8-Pad11) -> COL8
- U1 pad 12: unconnected-(U1-GPIO9-Pad12) -> COL9
- U1 pad 14: unconnected-(U1-GPIO10-Pad14) -> COL10
- U1 pad 15: unconnected-(U1-GPIO11-Pad15) -> COL11
- U1 pad 16: unconnected-(U1-GPIO12-Pad16) -> COL12
- U1 pad 17: unconnected-(U1-GPIO13-Pad17) -> COL13
- U1 pad 19: unconnected-(U1-GPIO14-Pad19) -> COL14
- U1 pad 2: unconnected-(U1-GPIO1-Pad2) -> COL1
- U1 pad 20: unconnected-(U1-GPIO15-Pad20) -> COL15
- U1 pad 21: unconnected-(U1-GPIO16-Pad21) -> COL16
- U1 pad 22: unconnected-(U1-GPIO17-Pad22) -> ROW0
- U1 pad 24: unconnected-(U1-GPIO18-Pad24) -> ROW1
- U1 pad 25: unconnected-(U1-GPIO19-Pad25) -> ROW2
- U1 pad 26: unconnected-(U1-GPIO20-Pad26) -> ROW3
- U1 pad 27: unconnected-(U1-GPIO21-Pad27) -> ROW4
- U1 pad 29: unconnected-(U1-GPIO22-Pad29) -> ROW5
- U1 pad 4: unconnected-(U1-GPIO2-Pad4) -> COL2
- U1 pad 5: unconnected-(U1-GPIO3-Pad5) -> COL3
- U1 pad 6: unconnected-(U1-GPIO4-Pad6) -> COL4
- U1 pad 7: unconnected-(U1-GPIO5-Pad7) -> COL5
- U1 pad 9: unconnected-(U1-GPIO6-Pad9) -> COL6
Routing:
- net COL1: track 0.00 -> 120.4 mm
- net COL2: track 0.00 -> 116.9 mm
- net COL13: track 0.00 -> 114.8 mm
- net COL0: track 0.00 -> 109.1 mm
- net COL3: track 0.00 -> 92.0 mm
- net COL4: track 0.00 -> 91.4 mm
- net COL5: track 0.00 -> 67.8 mm
- net COL8: track 0.00 -> 25.4 mm
- net COL9: track 0.00 -> 25.3 mm
- net COL11: track 0.00 -> 25.2 mm
- net COL10: track 0.00 -> 25.1 mm
- net COL12: track 0.00 -> 25.0 mm
- net COL7: track 0.00 -> 25.0 mm
- net COL6: track 0.00 -> 24.5 mm

Commit message: Finish column routing
Parts:
- moved U1 7.95 mm to (353.6, 40.1)
Connections:
- SW72 pad 1: COL8 -> COL9
- SW73 pad 1: COL9 -> COL10
- SW74 pad 1: COL10 -> COL11
Routing:
- net COL11: track 25.2 -> 114.2 mm
- net COL9: track 25.3 -> 112.8 mm
- net COL10: track 25.1 -> 112.1 mm
- net COL16: track 0.00 -> 78.5 mm
- net COL15: track 0.00 -> 78.4 mm
- net COL14: track 0.00 -> 77.7 mm
- net COL8: track 25.4 -> 92.4 mm
- net COL7: track 25.0 -> 92.0 mm
- net COL6: track 24.5 -> 91.5 mm
- net COL5: track 67.8 -> 111.8 mm
- net COL12: track 25.0 -> 48.0 mm
