File: PCB/_autosave-aniboard.kicad_pcb (KiCad board)
At the start: 2 copper layers, 365.5 x 216.7 mm, 198 parts, among them SW1 SW_Push, SW10 SW_Push, SW11 SW_Push, SW12 SW_Push, SW13 SW_Push, SW14 SW_Push, SW15 SW_Push, SW16 SW_Push, SW17 SW_Push, SW18 SW_Push, SW19 SW_Push, SW2 SW_Push, SW20 SW_Push, SW21 SW_Push, SW22 SW_Push, SW23 SW_Push, SW24 SW_Push, SW25 SW_Push, SW26 SW_Push, SW27 SW_Push, SW28 SW_Push, SW29 SW_Push, SW3 SW_Push, SW30 SW_Push, SW31 SW_Push, SW32 SW_Push, SW33 SW_Push, SW34 SW_Push, SW35 SW_Push, SW36 SW_Push, SW37 SW_Push, SW38 SW_Push, SW39 SW_Push, SW4 SW_Push, SW40 SW_Push, SW41 SW_Push, SW42 SW_Push, SW43 SW_Push, SW44 SW_Push, SW45 SW_Push, SW46 SW_Push, SW47 SW_Push, SW48 SW_Push, SW49 SW_Push, SW5 SW_Push, SW50 SW_Push, SW51 SW_Push, SW52 SW_Push, SW53 SW_Push, SW54 SW_Push, SW55 SW_Push, SW56 SW_Push, SW57 SW_Push, SW58 SW_Push, SW59 SW_Push, SW6 SW_Push, SW60 SW_Push, SW61 SW_Push, SW62 SW_Push, SW63 SW_Push, SW64 SW_Push, SW65 SW_Push, SW66 SW_Push, SW67 SW_Push, SW68 SW_Push, SW69 SW_Push, SW7 SW_Push, SW70 SW_Push, SW71 SW_Push, SW72 SW_Push, SW73 SW_Push, SW74 SW_Push, SW75 SW_Push, SW76 SW_Push, SW77 SW_Push, SW78 SW_Push, SW79 SW_Push, SW8 SW_Push, SW80 SW_Push, SW81 SW_Push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

Commit message: More keyboard
Parts:
- added LED15: MX_SK6812MINI-E, PCM_marbastlib-mx:LED_MX_6028R, F.Cu at (144.4, 185.3)
- added LED16: MX_SK6812MINI-E, PCM_marbastlib-mx:LED_MX_6028R, F.Cu at (144.4, 190.4)
- added LED17: MX_SK6812MINI-E, PCM_marbastlib-mx:LED_MX_6028R, F.Cu at (144.4, 195.4)
- added LED18: MX_SK6812MINI-E, PCM_marbastlib-mx:LED_MX_6028R, F.Cu at (144.4, 200.5)
- added LED19: MX_SK6812MINI-E, PCM_marbastlib-mx:LED_MX_6028R, F.Cu at (144.4, 205.5)
- added LED20: MX_SK6812MINI-E, PCM_marbastlib-mx:LED_MX_6028R, F.Cu at (144.4, 210.6)
- added LED21: MX_SK6812MINI-E, PCM_marbastlib-mx:LED_MX_6028R, F.Cu at (144.4, 215.6)
- added LED22: MX_SK6812MINI-E, PCM_marbastlib-mx:LED_MX_6028R, F.Cu at (153.3, 185.3)
- added LED23: MX_SK6812MINI-E, PCM_marbastlib-mx:LED_MX_6028R, F.Cu at (153.3, 190.4)
- added LED24: MX_SK6812MINI-E, PCM_marbastlib-mx:LED_MX_6028R, F.Cu at (153.3, 195.4)
- added LED25: MX_SK6812MINI-E, PCM_marbastlib-mx:LED_MX_6028R, F.Cu at (153.3, 200.5)
- added LED26: MX_SK6812MINI-E, PCM_marbastlib-mx:LED_MX_6028R, F.Cu at (153.3, 205.5)
- added LED27: MX_SK6812MINI-E, PCM_marbastlib-mx:LED_MX_6028R, F.Cu at (153.3, 210.6)
- added LED28: MX_SK6812MINI-E, PCM_marbastlib-mx:LED_MX_6028R, F.Cu at (153.3, 215.6)
- added LED29: MX_SK6812MINI-E, PCM_marbastlib-mx:LED_MX_6028R, F.Cu at (162.1, 185.3)
- added LED30: MX_SK6812MINI-E, PCM_marbastlib-mx:LED_MX_6028R, F.Cu at (162.1, 190.4)
- added LED31: MX_SK6812MINI-E, PCM_marbastlib-mx:LED_MX_6028R, F.Cu at (162.1, 195.4)
- added LED32: MX_SK6812MINI-E, PCM_marbastlib-mx:LED_MX_6028R, F.Cu at (162.1, 200.5)
- added LED33: MX_SK6812MINI-E, PCM_marbastlib-mx:LED_MX_6028R, F.Cu at (162.1, 205.5)
- added LED34: MX_SK6812MINI-E, PCM_marbastlib-mx:LED_MX_6028R, F.Cu at (162.1, 210.6)
- added LED35: MX_SK6812MINI-E, PCM_marbastlib-mx:LED_MX_6028R, F.Cu at (162.1, 215.6)
- added LED36: MX_SK6812MINI-E, PCM_marbastlib-mx:LED_MX_6028R, F.Cu at (171.0, 185.3)
- added LED37: MX_SK6812MINI-E, PCM_marbastlib-mx:LED_MX_6028R, F.Cu at (171.0, 190.4)
- added LED38: MX_SK6812MINI-E, PCM_marbastlib-mx:LED_MX_6028R, F.Cu at (171.0, 195.4)
- added LED39: MX_SK6812MINI-E, PCM_marbastlib-mx:LED_MX_6028R, F.Cu at (171.0, 200.5)
- added LED40: MX_SK6812MINI-E, PCM_marbastlib-mx:LED_MX_6028R, F.Cu at (171.0, 205.5)
- added LED41: MX_SK6812MINI-E, PCM_marbastlib-mx:LED_MX_6028R, F.Cu at (171.0, 210.6)
- added LED42: MX_SK6812MINI-E, PCM_marbastlib-mx:LED_MX_6028R, F.Cu at (171.0, 215.6)
- added LED43: MX_SK6812MINI-E, PCM_marbastlib-mx:LED_MX_6028R, F.Cu at (179.9, 185.3)
- added LED44: MX_SK6812MINI-E, PCM_marbastlib-mx:LED_MX_6028R, F.Cu at (179.9, 190.4)
- added LED45: MX_SK6812MINI-E, PCM_marbastlib-mx:LED_MX_6028R, F.Cu at (179.9, 195.4)
- added LED46: MX_SK6812MINI-E, PCM_marbastlib-mx:LED_MX_6028R, F.Cu at (179.9, 200.5)
- added LED47: MX_SK6812MINI-E, PCM_marbastlib-mx:LED_MX_6028R, F.Cu at (179.9, 205.5)
- added LED48: MX_SK6812MINI-E, PCM_marbastlib-mx:LED_MX_6028R, F.Cu at (179.9, 210.6)
- added LED49: MX_SK6812MINI-E, PCM_marbastlib-mx:LED_MX_6028R, F.Cu at (179.9, 215.6)
- added LED50: MX_SK6812MINI-E, PCM_marbastlib-mx:LED_MX_6028R, F.Cu at (188.7, 185.3)
- added LED51: MX_SK6812MINI-E, PCM_marbastlib-mx:LED_MX_6028R, F.Cu at (188.7, 190.4)
- added LED52: MX_SK6812MINI-E, PCM_marbastlib-mx:LED_MX_6028R, F.Cu at (188.7, 195.4)
- added LED53: MX_SK6812MINI-E, PCM_marbastlib-mx:LED_MX_6028R, F.Cu at (188.7, 200.5)
- added LED54: MX_SK6812MINI-E, PCM_marbastlib-mx:LED_MX_6028R, F.Cu at (188.7, 205.5)
- added LED55: MX_SK6812MINI-E, PCM_marbastlib-mx:LED_MX_6028R, F.Cu at (188.7, 210.6)
- moved D15 164.6 mm to (92.8, 81.3)
- moved D16 164.6 mm to (89.3, 81.3)
- moved D17 164.6 mm to (85.7, 81.3)
- moved D18 164.6 mm to (82.2, 81.3)
- moved D19 123.0 mm to (115.2, 211.3)
- moved D24 123.0 mm to (97.4, 211.3)
- moved D29 123.0 mm to (79.7, 211.3)
- moved D37 123.0 mm to (115.2, 200.5)
- moved D42 123.0 mm to (97.4, 200.5)
- moved D47 123.0 mm to (79.7, 200.5)
- moved D55 123.0 mm to (115.2, 189.7)
- moved D60 123.0 mm to (97.4, 189.7)
- moved D65 123.0 mm to (79.7, 189.7)
- moved D73 123.0 mm to (115.2, 179.0)
- moved D78 123.0 mm to (97.4, 179.0)
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Connections:
- LED14 pad 3: unconnected-(LED14-DIN-Pad3) -> LED1
- U1 pad 21: COL16 -> ROW0
- U1 pad 22: ROW0 -> COL16
