File: PCB/aniboard.kicad_sch (KiCad schematic)
At the start: 151 parts, among them SW1 SW_Push, SW10 SW_Push, SW11 SW_Push, SW12 SW_Push, SW13 SW_Push, SW14 SW_Push, SW15 SW_Push, SW16 SW_Push, SW17 SW_Push, SW18 SW_Push, SW19 SW_Push, SW2 SW_Push, SW20 SW_Push, SW21 SW_Push, SW22 SW_Push, SW23 SW_Push, SW24 SW_Push, SW25 SW_Push, SW26 SW_Push, SW27 SW_Push, SW28 SW_Push, SW29 SW_Push, SW3 SW_Push, SW30 SW_Push, SW31 SW_Push, SW32 SW_Push, SW33 SW_Push, SW34 SW_Push, SW35 SW_Push, SW36 SW_Push, SW37 SW_Push, SW38 SW_Push, SW39 SW_Push, SW4 SW_Push, SW40 SW_Push, SW41 SW_Push, SW42 SW_Push, SW43 SW_Push, SW44 SW_Push, SW45 SW_Push, SW46 SW_Push, SW47 SW_Push, SW48 SW_Push, SW49 SW_Push, SW5 SW_Push, SW50 SW_Push, SW51 SW_Push, SW52 SW_Push, SW53 SW_Push, SW54 SW_Push, SW55 SW_Push, SW56 SW_Push, SW57 SW_Push, SW58 SW_Push, SW59 SW_Push, SW6 SW_Push, SW60 SW_Push, SW61 SW_Push, SW62 SW_Push, SW63 SW_Push, SW64 SW_Push, SW65 SW_Push, SW66 SW_Push, SW67 SW_Push, SW68 SW_Push, SW69 SW_Push, SW7 SW_Push, SW70 SW_Push, SW71 SW_Push, SW72 SW_Push, SW73 SW_Push, SW74 SW_Push, SW75 SW_Push, SW8 SW_Push, SW9 SW_Push, U1 Pico

Commit message: First three rows
Parts:
- added D76, D77, D78, D79, D80, D81, D82, D83, D84, D85, D86, D87, D88: D, symbol Device:D
- added S1: MX_stab, PCM_marbastlib-mx:STAB_MX_P_2u, symbol PCM_marbastlib-mx:MX_stab
- added SW76, SW77, SW78, SW79, SW80, SW81, SW82, SW83, SW84, SW85, SW86, SW87, SW88: SW_Push, symbol Switch:SW_Push
- SW1, SW14, SW29, SW42: footprint (none) -> PCM_marbastlib-mx:SW_MX_1.5u
- SW10, SW11, SW12, SW13, SW15, SW16, SW17, SW18, SW19, SW2, SW20, SW21, SW22, SW23, SW24, SW25, SW26, SW27, SW28, SW3, SW30, SW31, SW32, SW33, SW34, SW35, SW36, SW37, SW38, SW39, SW4, SW40, SW41, SW5, SW6, SW7, SW8, SW9: footprint (none) -> PCM_marbastlib-mx:SW_MX_1u
Connections:
- net COL8: now reaches SW23.1, SW37.1, SW51.1, SW64.1, SW72.1, SW9.1
- net ROW3: now reaches D43.1 (K), D44.1 (K), D45.1 (K), D46.1 (K), D47.1 (K), D48.1 (K), D49.1 (K), D50.1 (K), D51.1 (K), D52.1 (K), D53.1 (K), D54.1 (K), D55.1 (K)
- net ROW3: now also D86.1 (K), D87.1 (K), D88.1 (K)
- net COL10: now reaches SW11.1, SW25.1, SW39.1, SW53.1, SW66.1, SW74.1
- net COL2: now reaches SW17.1, SW3.1, SW31.1, SW45.1, SW58.1, SW70.1
- net COL5: now reaches SW20.1, SW34.1, SW48.1, SW6.1, SW61.1, SW71.1
- net COL9: now reaches SW10.1, SW24.1, SW38.1, SW52.1, SW65.1, SW73.1
- net COL11: now reaches SW12.1, SW26.1, SW40.1, SW54.1, SW67.1, SW75.1
- net ROW0: now reaches D1.1 (K), D10.1 (K), D11.1 (K), D12.1 (K), D13.1 (K), D14.1 (K), D2.1 (K), D3.1 (K), D4.1 (K), D5.1 (K), D6.1 (K), D7.1 (K), D8.1 (K), D9.1 (K)
- net ROW2: now reaches D29.1 (K), D30.1 (K), D31.1 (K), D32.1 (K), D33.1 (K), D34.1 (K), D35.1 (K), D36.1 (K), D37.1 (K), D38.1 (K), D39.1 (K), D40.1 (K), D41.1 (K), D42.1 (K)
- net ROW2: now also D83.1 (K), D84.1 (K), D85.1 (K)
- net ROW4: now reaches D56.1 (K), D57.1 (K), D58.1 (K), D59.1 (K), D60.1 (K), D61.1 (K), D62.1 (K), D63.1 (K), D64.1 (K), D65.1 (K), D66.1 (K), D67.1 (K)
- net ROW4: now also D79.1 (K)
- net COL3: now reaches SW18.1
- net COL3: now also SW32.1, SW4.1, SW46.1, SW59.1
- net COL13: now reaches SW14.1
- net COL13: now also SW28.1, SW42.1
- net COL1: now reaches SW16.1, SW2.1, SW30.1, SW44.1, SW57.1, SW69.1
- net ROW1: now reaches D15.1 (K), D16.1 (K), D17.1 (K), D18.1 (K), D19.1 (K), D20.1 (K), D21.1 (K), D22.1 (K), D23.1 (K), D24.1 (K), D25.1 (K), D26.1 (K), D27.1 (K), D28.1 (K)
- net ROW1: now also D80.1 (K), D81.1 (K), D82.1 (K)
- net COL4: now reaches SW33.1
- net COL4: now also SW19.1, SW47.1, SW5.1, SW60.1
- net COL0: now reaches SW1.1, SW15.1, SW29.1, SW43.1, SW56.1, SW68.1
- net COL7: now reaches SW50.1
- net COL7: now also SW22.1, SW36.1, SW63.1, SW8.1
- net ROW5: now reaches D68.1 (K), D69.1 (K), D70.1 (K), D71.1 (K), D72.1 (K), D73.1 (K), D74.1 (K), D75.1 (K)
- net ROW5: now also D76.1 (K), D77.1 (K), D78.1 (K)
- net COL6: now reaches SW49.1
- net COL6: now also SW21.1, SW35.1, SW62.1, SW7.1
- net COL12: now reaches SW13.1
- net COL12: now also SW27.1, SW41.1, SW55.1
- new net: D85.2 (A), SW85.2
- new net: D81.2 (A), SW81.2
- new net: D82.2 (A), SW82.2
- new net: D88.2 (A), SW88.2
- new net: D83.2 (A), SW83.2
- new net: D79.2 (A), SW79.2
- new net: D80.2 (A), SW80.2
- new net: D86.2 (A), SW86.2
- new net: D76.2 (A), SW76.2
- new net: D84.2 (A), SW84.2
- new net: D77.2 (A), SW77.2
- new net: D87.2 (A), SW87.2
- new net: D78.2 (A), SW78.2
- new net COL14: SW76.1, SW80.1, SW83.1, SW86.1
- new net COL15: SW77.1, SW79.1, SW81.1, SW84.1, SW87.1
- new net COL16: SW78.1, SW82.1, SW85.1, SW88.1
Other:
- moved on the sheet: U1

Commit message: Keyboard layout
Parts:
- added S2, S3: MX_stab, PCM_marbastlib-mx:STAB_MX_2.25u, symbol PCM_marbastlib-mx:MX_stab
- added S4: MX_stab, PCM_marbastlib-mx:STAB_MX_2.75u, symbol PCM_marbastlib-mx:MX_stab
- added S5: MX_stab, PCM_marbastlib-mx:STAB_MX_6.25u, symbol PCM_marbastlib-mx:MX_stab
- S1: footprint PCM_marbastlib-mx:STAB_MX_P_2u -> PCM_marbastlib-mx:STAB_MX_2u
- SW43: footprint (none) -> PCM_marbastlib-mx:SW_MX_1.75u
- SW44, SW45, SW46, SW47, SW48, SW49, SW50, SW51, SW52, SW53, SW54, SW55, SW56, SW57, SW58, SW59, SW60, SW61, SW62, SW63, SW64, SW65, SW66, SW67, SW71, SW76, SW77, SW78, SW79, SW80, SW81, SW82, SW83, SW84, SW85, SW86, SW87, SW88: footprint (none) -> PCM_marbastlib-mx:SW_MX_1u
- SW68, SW69, SW70, SW72, SW73, SW74, SW75: footprint (none) -> PCM_marbastlib-mx:SW_MX_1.25u

Commit message: Continue routing PCB
Parts:
- D1, D10, D11, D12, D13, D14, D15, D16, D17, D18, D19, D2, D20, D21, D22, D23, D24, D25, D26, D27, D28, D29, D3, D30, D31, D32, D33, D34, D35, D36, D37, D38, D39, D4, D40, D41, D42, D43, D44, D45, D46, D47, D48, D49, D5, D50, D51, D52, D53, D54, D55, D56, D57, D58, D59, D6, D60, D61, D62, D63, D64, D65, D66, D67, D68, D69, D7, D70, D71, D72, D73, D74, D75, D76, D77, D78, D79, D8, D80, D81, D82, D83, D84, D85, D86, D87, D88, D9: footprint (none) -> Diode_THT:D_DO-35_SOD27_P7.62mm_Horizontal
Connections:
- net COL0: now also U1.1 (GPIO0)
- net COL1: now also U1.2 (GPIO1)
- net COL10: now also U1.14 (GPIO10)
- net COL11: now also U1.15 (GPIO11); no longer SW67.1, SW75.1
- net COL12: now also U1.16 (GPIO12); no longer SW55.1
- net COL13: now also SW55.1, SW67.1, SW75.1, U1.17 (GPIO13)
- net COL14: now also U1.19 (GPIO14)
- net COL15: now also U1.20 (GPIO15)
- net COL16: now also U1.21 (GPIO16)
- net COL2: now also U1.4 (GPIO2)
- net COL3: now also U1.5 (GPIO3)
- net COL4: now also U1.6 (GPIO4)
- net COL5: now also U1.7 (GPIO5)
- net COL6: now also U1.9 (GPIO6)
- net COL7: now also U1.10 (GPIO7)
- net COL8: now also U1.11 (GPIO8)
- net COL9: now also U1.12 (GPIO9)
- net ROW0: now also U1.22 (GPIO17)
- net ROW1: now also U1.24 (GPIO18)
- net ROW2: now also U1.25 (GPIO19)
- net ROW3: now also U1.26 (GPIO20); no longer D55.1 (K)
- net ROW4: now also U1.27 (GPIO21)
- net ROW5: now also U1.29 (GPIO22)
Other:
- moved on the sheet: D55, D67, D75, S2, S4, SW55, SW67, SW75

Commit message: Finish column routing
Connections:
- net COL10: now also SW73.1; no longer SW74.1
- net COL11: now also SW74.1
- net COL8: no longer SW72.1
- net COL9: now also SW72.1; no longer SW73.1
Other:
- moved on the sheet: D72, D73, D74, SW72, SW73, SW74
Changed lines of the file:
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@@
 	)
 	(junction
-		(at 173.99 123.19)
-		(diameter 0)
-		(color 0 0 0 0)
-	)
-	(junction
 		(at 184.15 48.26)
 		(diameter 0)
@@
 	)
 	(junction
+		(at 223.52 101.6)
+		(diameter 0)
+		(color 0 0 0 0)
+	)
+	(junction
 		(at 68.58 88.9)
 		(diameter 0)
@@
 	)
 	(junction
-		(at 184.15 151.13)
-		(diameter 0)
-		(color 0 0 0 0)
-	)
-	(junction
 		(at 167.64 88.9)
 		(diameter 0)
@@
 	)
 	(junction
+		(at 233.68 151.13)
+		(diameter 0)
+		(color 0 0 0 0)
+	)
+	(junction
 		(at 91.44 81.28)
 		(diameter 0)
@@
 	(wire
 		(pts
-			(xy 184.15 151.13) (xy 200.66 151.13)
-		)
-		(stroke
-			(width 0)
-			(type default)
-		)
-	)
-	(wire
-		(pts
 			(xy 217.17 109.22) (xy 233.68 109.22)
 		)
@@
 	(wire
 		(pts
-			(xy 190.5 123.19) (xy 190.5 143.51)
+			(xy 207.01 123.19) (xy 207.01 143.51)
 		)
 		(stroke
@@
 	(wire
 		(pts
-			(xy 207.01 123.19) (xy 207.01 143.51)
+			(xy 223.52 101.6) (xy 223.52 143.51)
 		)
 		(stroke
@@
 	(wire
 		(pts
+			(xy 233.68 151.13) (xy 266.7 151.13)
+		)
+		(stroke
+			(width 0)
+			(type default)
+		)
+	)
+	(wire
+		(pts
 			(xy 74.93 30.48) (xy 74.93 40.64)
 		)
@@
 	(wire
 		(pts
-			(xy 173.99 123.19) (xy 173.99 143.51)
+			(xy 190.5 123.19) (xy 190.5 143.51)
 		)
 		(stroke
@@
 	(wire
 		(pts
-			(xy 217.17 151.13) (xy 266.7 151.13)
+			(xy 217.17 151.13) (xy 233.68 151.13)
 		)
 		(stroke
@@
 	(wire
 		(pts
-			(xy 134.62 151.13) (xy 184.15 151.13)
+			(xy 134.62 151.13) (xy 200.66 151.13)
 		)
 		(stroke
@@
 	(symbol
 		(lib_id "Switch:SW_Push")
-		(at 195.58 143.51 0)
+		(at 212.09 143.51 0)
 		(unit 1)
 		(exclude_from_sim no)
@@
 		(fields_autoplaced yes)
 		(property "Reference" "SW73"
-			(at 195.58 135.89 0)
+			(at 212.09 135.89 0)
 			(effects
 				(font
@@
 		)
 		(property "Value" "SW_Push"
-			(at 195.58 138.43 0)
+			(at 212.09 138.43 0)
 			(effects
 				(font
@@
 		)
 		(property "Footprint" "PCM_marbastlib-mx:SW_MX_1.25u"
-			(at 195.58 138.43 0)
+			(at 212.09 138.43 0)
 			(effects
 				(font
@@
 		)
 		(property "Datasheet" "~"
-			(at 195.58 138.43 0)
+			(at 212.09 138.43 0)
 			(effects
 				(font
@@
 		)
 		(property "Description" "Push button switch, generic, two pins"
-			(at 195.58 143.51 0)
+			(at 212.09 143.51 0)
 			(effects
 				(font
@@
 	(symbol
 		(lib_id "Device:D")
-		(at 200.66 147.32 90)
+		(at 217.17 147.32 90)
 		(unit 1)
 		(exclude_from_sim no)
@@
 		(fields_autoplaced yes)
 		(property "Reference" "D73"
-			(at 203.2 146.0499 90)
+			(at 219.71 146.0499 90)
 			(effects
 				(font
@@
 		)
 		(property "Value" "D"
-			(at 203.2 148.5899 90)
+			(at 219.71 148.5899 90)
 			(effects
 				(font
@@
 		)
 		(property "Footprint" "Diode_THT:D_DO-35_SOD27_P7.62mm_Horizontal"
-			(at 200.66 147.32 0)
+			(at 217.17 147.32 0)
 			(effects
 				(font
@@
 		)
 		(property "Datasheet" "~"
-			(at 200.66 147.32 0)
+			(at 217.17 147.32 0)
 			(effects
 				(font
@@
 		)
 		(property "Description" "Diode"
-			(at 200.66 147.32 0)
+			(at 217.17 147.32 0)
 			(effects
 				(font
@@
 		)
 		(property "Sim.Device" "D"
-			(at 200.66 147.32 0)
+			(at 217.17 147.32 0)
 			(effects
 				(font
@@
 		)
 		(property "Sim.Pins" "1=K 2=A"
-			(at 200.66 147.32 0)
+			(at 217.17 147.32 0)
 			(effects
 				(font
@@
 	(symbol
 		(lib_id "Device:D")
-		(at 217.17 147.32 90)
+		(at 233.68 147.32 90)
 		(unit 1)
 		(exclude_from_sim no)
@@
 		(fields_autoplaced yes)
 		(property "Reference" "D74"
-			(at 219.71 146.0499 90)
+			(at 236.22 146.0499 90)
 			(effects
 				(font
@@
 		)
 		(property "Value" "D"
-			(at 219.71 148.5899 90)
+			(at 236.22 148.5899 90)
 			(effects
 				(font
@@
 		)
 		(property "Footprint" "Diode_THT:D_DO-35_SOD27_P7.62mm_Horizontal"
-			(at 217.17 147.32 0)
+			(at 233.68 147.32 0)
 			(effects
 				(font
@@
 		)
 		(property "Datasheet" "~"
-			(at 217.17 147.32 0)
+			(at 233.68 147.32 0)
 			(effects
 				(font
@@
 		)
 		(property "Description" "Diode"
-			(at 217.17 147.32 0)
+			(at 233.68 147.32 0)
 			(effects
 				(font
@@
 		)
 		(property "Sim.Device" "D"
-			(at 217.17 147.32 0)
+			(at 233.68 147.32 0)
 			(effects
 				(font
@@
 		)
 		(property "Sim.Pins" "1=K 2=A"
-			(at 217.17 147.32 0)
+			(at 233.68 147.32 0)
 			(effects
 				(font
@@
 	(symbol
 		(lib_id "Device:D")
-		(at 184.15 147.32 90)
+		(at 200.66 147.32 90)
 		(unit 1)
 		(exclude_from_sim no)
@@
 		(fields_autoplaced yes)
 		(property "Reference" "D72"
-			(at 186.69 146.0499 90)
+			(at 203.2 146.0499 90)
 			(effects
 				(font
@@
 		)
 		(property "Value" "D"
-			(at 186.69 148.5899 90)
+			(at 203.2 148.5899 90)
 			(effects
 				(font
@@
 		)
 		(property "Footprint" "Diode_THT:D_DO-35_SOD27_P7.62mm_Horizontal"
-			(at 184.15 147.32 0)
+			(at 200.66 147.32 0)
 			(effects
 				(font
@@
 		)
 		(property "Datasheet" "~"
-			(at 184.15 147.32 0)
+			(at 200.66 147.32 0)
 			(effects
 				(font
@@
 		)
 		(property "Description" "Diode"
-			(at 184.15 147.32 0)
+			(at 200.66 147.32 0)
 			(effects
 				(font
@@
 		)
 		(property "Sim.Device" "D"
-			(at 184.15 147.32 0)
+			(at 200.66 147.32 0)
 			(effects
 				(font
@@
 		)
 		(property "Sim.Pins" "1=K 2=A"
-			(at 184.15 147.32 0)
+			(at 200.66 147.32 0)
 			(effects
 				(font
@@
 	(symbol
 		(lib_id "Switch:SW_Push")
-		(at 179.07 143.51 0)
+		(at 195.58 143.51 0)
 		(unit 1)
 		(exclude_from_sim no)
@@
 		(fields_autoplaced yes)
 		(property "Reference" "SW72"
-			(at 179.07 135.89 0)
+			(at 195.58 135.89 0)
 			(effects
 				(font
@@
 		)
 		(property "Value" "SW_Push"
-			(at 179.07 138.43 0)
+			(at 195.58 138.43 0)
 			(effects
 				(font
@@
 		)
 		(property "Footprint" "PCM_marbastlib-mx:SW_MX_1.25u"
-			(at 179.07 138.43 0)
+			(at 195.58 138.43 0)
 			(effects
 				(font
@@
 		)
 		(property "Datasheet" "~"
-			(at 179.07 138.43 0)
+			(at 195.58 138.43 0)
 			(effects
 				(font
@@
 		)
 		(property "Description" "Push button switch, generic, two pins"
-			(at 179.07 143.51 0)
+			(at 195.58 143.51 0)
 			(effects
 				(font
@@
 	(symbol
 		(lib_id "Switch:SW_Push")
-		(at 212.09 143.51 0)
+		(at 228.6 143.51 0)
 		(unit 1)
 		(exclude_from_sim no)
@@
 		(fields_autoplaced yes)
 		(property "Reference" "SW74"
-			(at 212.09 135.89 0)
+			(at 228.6 135.89 0)
 			(effects
 				(font
@@
 		)
 		(property "Value" "SW_Push"
-			(at 212.09 138.43 0)
+			(at 228.6 138.43 0)
 			(effects
 				(font
@@
 		)
 		(property "Footprint" "PCM_marbastlib-mx:SW_MX_1.25u"
-			(at 212.09 138.43 0)
+			(at 228.6 138.43 0)
 			(effects
 				(font
@@
 		)
 		(property "Datasheet" "~"
-			(at 212.09 138.43 0)
+			(at 228.6 138.43 0)
 			(effects
 				(font
@@
 		)
 		(property "Description" "Push button switch, generic, two pins"
-			(at 212.09 143.51 0)
+			(at 228.6 143.51 0)
 			(effects
 				(font

Commit message: More keyboard
Parts:
- added JP1: SolderJumper_2_Bridged, Jumper:SolderJumper-2_P1.3mm_Bridged_RoundedPad1.0x1.5mm, symbol Jumper:SolderJumper_2_Bridged
- added JP2: SolderJumper_2_Open, Jumper:SolderJumper-2_P1.3mm_Open_RoundedPad1.0x1.5mm, symbol Jumper:SolderJumper_2_Open
- added LED1, LED10, LED11, LED12, LED13, LED14, LED15, LED16, LED17, LED18, LED19, LED2, LED20, LED21, LED22, LED23, LED24, LED25, LED26, LED27, LED28, LED29, LED3, LED30, LED31, LED32, LED33, LED34, LED35, LED36, LED37, LED38, LED39, LED4, LED40, LED41, LED42, LED43, LED44, LED45, LED46, LED47, LED48, LED49, LED5, LED50, LED51, LED52, LED53, LED54, LED55, LED56, LED57, LED58, LED59, LED6, LED60, LED61, LED62, LED63, LED64, LED65, LED66, LED67, LED68, LED69, LED7, LED70, LED71, LED72, LED73, LED74, LED75, LED76, LED77, LED78, LED79, LED8, LED80, LED81, LED82, LED83, LED84, LED85, LED86, LED87, LED88, LED9: MX_SK6812MINI-E, PCM_marbastlib-mx:LED_MX_6028R, symbol PCM_marbastlib-mx:MX_SK6812MINI-E
- D1, D10, D11, D12, D13, D14, D15, D16, D17, D18, D19, D2, D20, D21, D22, D23, D24, D25, D26, D27, D28, D29, D3, D30, D31, D32, D33, D34, D35, D36, D37, D38, D39, D4, D40, D41, D42, D43, D44, D45, D46, D47, D48, D49, D5, D50, D51, D52, D53, D54, D55, D56, D57, D58, D59, D6, D60, D61, D62, D63, D64, D65, D66, D67, D68, D69, D7, D70, D71, D72, D73, D74, D75, D76, D77, D78, D79, D8, D80, D81, D82, D83, D84, D85, D86, D87, D88, D9: footprint Diode_THT:D_DO-35_SOD27_P7.62mm_Horizontal -> Diode_SMD:D_MiniMELF_Handsoldering
Connections:
- net COL16: now also U1.22 (GPIO17); no longer U1.21 (GPIO16)
- net ROW0: now also U1.21 (GPIO16); no longer U1.22 (GPIO17)
- net GND: now reaches U1.13 (GND)
- net GND: now also U1.18 (GND), U1.23 (GND), U1.28 (GND), U1.3 (GND), U1.38 (GND), U1.8 (GND), LED1.4 (VSS), LED10.4 (VSS), LED11.4 (VSS), LED12.4 (VSS), LED13.4 (VSS), LED14.4 (VSS), LED15.4 (VSS), LED16.4 (VSS), LED17.4 (VSS), LED18.4 (VSS), LED19.4 (VSS), LED2.4 (VSS), LED20.4 (VSS), LED21.4 (VSS), LED22.4 (VSS), LED23.4 (VSS), LED24.4 (VSS), LED25.4 (VSS), LED26.4 (VSS), LED27.4 (VSS), LED28.4 (VSS), LED29.4 (VSS), LED3.4 (VSS), LED30.4 (VSS), LED31.4 (VSS), LED32.4 (VSS), LED33.4 (VSS), LED34.4 (VSS), LED35.4 (VSS), LED36.4 (VSS), LED37.4 (VSS), LED38.4 (VSS), LED39.4 (VSS), LED4.4 (VSS), LED40.4 (VSS), LED41.4 (VSS), LED42.4 (VSS), LED43.4 (VSS), LED44.4 (VSS), LED45.4 (VSS), LED46.4 (VSS), LED47.4 (VSS), LED48.4 (VSS), LED49.4 (VSS), LED5.4 (VSS), LED50.4 (VSS), LED51.4 (VSS), LED52.4 (VSS), LED53.4 (VSS), LED54.4 (VSS), LED55.4 (VSS), LED56.4 (VSS), LED57.4 (VSS), LED58.4 (VSS), LED59.4 (VSS), LED6.4 (VSS), LED60.4 (VSS), LED61.4 (VSS), LED62.4 (VSS), LED63.4 (VSS), LED64.4 (VSS), LED65.4 (VSS), LED66.4 (VSS), LED67.4 (VSS), LED68.4 (VSS), LED69.4 (VSS), LED7.4 (VSS), LED70.4 (VSS), LED71.4 (VSS), LED72.4 (VSS), LED73.4 (VSS), LED74.4 (VSS), LED75.4 (VSS), LED76.4 (VSS), LED77.4 (VSS), LED78.4 (VSS), LED79.4 (VSS), LED8.4 (VSS), LED80.4 (VSS), LED81.4 (VSS), LED82.4 (VSS), LED83.4 (VSS), LED84.4 (VSS), LED85.4 (VSS), LED86.4 (VSS), LED87.4 (VSS), LED88.4 (VSS), LED9.4 (VSS)
- net at U1.39 (VSYS): now also JP2.1 (A)
- net at U1.40 (VBUS): now also JP1.1 (A)
- new net: LED86.3 (DIN), LED87.2 (DOUT)
- new net: LED87.3 (DIN), LED88.2 (DOUT)
- new net: LED32.3 (DIN), LED33.2 (DOUT)
- new net: LED33.3 (DIN), LED34.2 (DOUT)
- new net: LED11.3 (DIN), LED12.2 (DOUT)
- new net: LED12.3 (DIN), LED13.2 (DOUT)
- new net: LED28.3 (DIN), LED80.2 (DOUT)
- new net: LED80.3 (DIN), LED81.2 (DOUT)
- new net: LED77.3 (DIN), LED78.2 (DOUT)
- new net: LED42.3 (DIN), LED83.2 (DOUT)
- new net: LED83.3 (DIN), LED84.2 (DOUT)
- new net: LED22.3 (DIN), LED23.2 (DOUT)
- new net: LED23.3 (DIN), LED24.2 (DOUT)
- new net: LED29.3 (DIN), LED30.2 (DOUT)
- new net: LED30.3 (DIN), LED31.2 (DOUT)
- new net: LED49.3 (DIN), LED50.2 (DOUT)
- new net: LED50.3 (DIN), LED51.2 (DOUT)
- new net: LED2.3 (DIN), LED3.2 (DOUT)
- new net: LED3.3 (DIN), LED4.2 (DOUT)
- new net: LED81.3 (DIN), LED82.2 (DOUT)
- new net: LED43.3 (DIN), LED44.2 (DOUT)
- new net: LED5.3 (DIN), LED6.2 (DOUT)
- new net: LED6.3 (DIN), LED7.2 (DOUT)
- new net: LED24.3 (DIN), LED25.2 (DOUT)
- new net: LED73.3 (DIN), LED74.2 (DOUT)
- new net: LED74.3 (DIN), LED75.2 (DOUT)
- new net: LED51.3 (DIN), LED52.2 (DOUT)
- new net: LED56.3 (DIN), LED57.2 (DOUT)
- new net: LED4.3 (DIN), LED5.2 (DOUT)
- new net: LED72.3 (DIN), LED73.2 (DOUT)
- new net: LED45.3 (DIN), LED46.2 (DOUT)
- new net: LED46.3 (DIN), LED47.2 (DOUT)
- new net: LED68.3 (DIN), LED69.2 (DOUT)
- new net: LED69.3 (DIN), LED70.2 (DOUT)
- new net: LED7.3 (DIN), LED8.2 (DOUT)
- new net: LED8.3 (DIN), LED9.2 (DOUT)
- new net: LED25.3 (DIN), LED26.2 (DOUT)
- new net: LED26.3 (DIN), LED27.2 (DOUT)
- new net: LED10.2 (DOUT), LED9.3 (DIN)
- new net: LED10.3 (DIN), LED11.2 (DOUT)
- new net: LED58.3 (DIN), LED59.2 (DOUT)
- new net: LED59.3 (DIN), LED60.2 (DOUT)
- new net: LED57.3 (DIN), LED58.2 (DOUT)
- new net: LED48.3 (DIN), LED49.2 (DOUT)
- new net: LED1.3 (DIN), LED2.2 (DOUT)
- new net: LED38.3 (DIN), LED39.2 (DOUT)
- new net: LED39.3 (DIN), LED40.2 (DOUT)
- new net: LED60.3 (DIN), LED61.2 (DOUT)
- new net: LED44.3 (DIN), LED45.2 (DOUT)
- new net: LED84.3 (DIN), LED85.2 (DOUT)
- new net: LED75.3 (DIN), LED76.2 (DOUT)
- new net: LED64.3 (DIN), LED65.2 (DOUT)
- new net: LED65.3 (DIN), LED66.2 (DOUT)
- new net: LED13.3 (DIN), LED14.2 (DOUT)
- new net: LED19.3 (DIN), LED20.2 (DOUT)
- new net: LED20.3 (DIN), LED21.2 (DOUT)
- new net: LED40.3 (DIN), LED41.2 (DOUT)
- new net: LED52.3 (DIN), LED53.2 (DOUT)
- new net: LED53.3 (DIN), LED54.2 (DOUT)
- new net: LED61.3 (DIN), LED62.2 (DOUT)
- new net: LED70.3 (DIN), LED71.2 (DOUT)
- new net: LED36.3 (DIN), LED37.2 (DOUT)
- new net: LED37.3 (DIN), LED38.2 (DOUT)
- new net: LED35.3 (DIN), LED36.2 (DOUT)
- new net: LED67.3 (DIN), LED79.2 (DOUT)
- new net: LED18.3 (DIN), LED19.2 (DOUT)
- new net: LED15.3 (DIN), LED16.2 (DOUT)
- new net: LED66.3 (DIN), LED67.2 (DOUT)
- new net: LED54.3 (DIN), LED55.2 (DOUT)
- new net: LED31.3 (DIN), LED32.2 (DOUT)
- new net: LED34.3 (DIN), LED35.2 (DOUT)
- new net: LED55.3 (DIN), LED86.2 (DOUT)
- new net: LED16.3 (DIN), LED17.2 (DOUT)
- new net: LED17.3 (DIN), LED18.2 (DOUT)
- new net: LED27.3 (DIN), LED28.2 (DOUT)
- new net: LED71.3 (DIN), LED72.2 (DOUT)
- new net: LED62.3 (DIN), LED63.2 (DOUT)
- new net: LED63.3 (DIN), LED64.2 (DOUT)
- new net: LED76.3 (DIN), LED77.2 (DOUT)
- new net: LED41.3 (DIN), LED42.2 (DOUT)
- new net: LED47.3 (DIN), LED48.2 (DOUT)
- new net: LED21.3 (DIN), LED22.2 (DOUT)
- new net +5V: JP1.2 (B), JP2.2 (B), LED1.1 (VDD), LED10.1 (VDD), LED11.1 (VDD), LED12.1 (VDD), LED13.1 (VDD), LED14.1 (VDD), LED15.1 (VDD), LED16.1 (VDD), LED17.1 (VDD), LED18.1 (VDD), LED19.1 (VDD), LED2.1 (VDD), LED20.1 (VDD), LED21.1 (VDD), LED22.1 (VDD), LED23.1 (VDD), LED24.1 (VDD), LED25.1 (VDD), LED26.1 (VDD), LED27.1 (VDD), LED28.1 (VDD), LED29.1 (VDD), LED3.1 (VDD), LED30.1 (VDD), LED31.1 (VDD), LED32.1 (VDD), LED33.1 (VDD), LED34.1 (VDD), LED35.1 (VDD), LED36.1 (VDD), LED37.1 (VDD), LED38.1 (VDD), LED39.1 (VDD), LED4.1 (VDD), LED40.1 (VDD), LED41.1 (VDD), LED42.1 (VDD), LED43.1 (VDD), LED44.1 (VDD), LED45.1 (VDD), LED46.1 (VDD), LED47.1 (VDD), LED48.1 (VDD), LED49.1 (VDD), LED5.1 (VDD), LED50.1 (VDD), LED51.1 (VDD), LED52.1 (VDD), LED53.1 (VDD), LED54.1 (VDD), LED55.1 (VDD), LED56.1 (VDD), LED57.1 (VDD), LED58.1 (VDD), LED59.1 (VDD), LED6.1 (VDD), LED60.1 (VDD), LED61.1 (VDD), LED62.1 (VDD), LED63.1 (VDD), LED64.1 (VDD), LED65.1 (VDD), LED66.1 (VDD), LED67.1 (VDD), LED68.1 (VDD), LED69.1 (VDD), LED7.1 (VDD), LED70.1 (VDD), LED71.1 (VDD), LED72.1 (VDD), LED73.1 (VDD), LED74.1 (VDD), LED75.1 (VDD), LED76.1 (VDD), LED77.1 (VDD), LED78.1 (VDD), LED79.1 (VDD), LED8.1 (VDD), LED80.1 (VDD), LED81.1 (VDD), LED82.1 (VDD), LED83.1 (VDD), LED84.1 (VDD), LED85.1 (VDD), LED86.1 (VDD), LED87.1 (VDD), LED88.1 (VDD), LED9.1 (VDD)
- new net LED: LED14.3 (DIN)
- new net LED1: LED1.2 (DOUT), LED82.3 (DIN)
- new net LED2: LED15.2 (DOUT), LED85.3 (DIN)
- new net LED3: LED29.2 (DOUT), LED43.2 (DOUT), LED88.3 (DIN)
- new net LED4: LED56.2 (DOUT), LED78.3 (DIN), LED79.3 (DIN)
Other:
- moved on the sheet: D1, D10, D11, D12, D13, D14, D15, D16, D17, D18, D19, D2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
